Commit message: feat: add create3 rgbd camera bridge

File: create3_sim/irobot_create_common/irobot_create_description/urdf/create3.urdf.xacro (robot description, xacro)
@@ -8,4 +8,5 @@
   <xacro:include filename="$(find irobot_create_description)/urdf/sensors/imu.urdf.xacro" />
   <xacro:include filename="$(find irobot_create_description)/urdf/sensors/lidar.urdf.xacro" />
+  <xacro:include filename="$(find irobot_create_description)/urdf/sensors/rgbd_camera.urdf.xacro" />
   <xacro:include filename="$(find irobot_create_description)/urdf/sensors/ir_intensity.urdf.xacro" />
   <xacro:include filename="$(find irobot_create_description)/urdf/sensors/ir_opcode_receivers.urdf.xacro" />
@@ -106,4 +107,8 @@
     <origin xyz="0.0 0.0 ${0.05 + base_link_z_offset}"/>
   </xacro:lidar_sensor>
+  <!-- Front RGB-D camera for semantic navigation experiments -->
+  <xacro:rgbd_camera_sensor gazebo="$(arg gazebo)" namespace="$(arg namespace)">
+    <origin xyz="0.135 0 ${0.135 + base_link_z_offset}" rpy="0 ${10*deg2rad} 0"/>
+  </xacro:rgbd_camera_sensor>
   <xacro:if value="${'$(arg gazebo)' == 'classic'}">
     <gazebo>

Commit message: feat: add lyra rgbd probe pipeline

File: create3_sim/irobot_create_common/irobot_create_description/urdf/create3.urdf.xacro (robot description, xacro)
@@ -109,5 +109,5 @@
   <!-- Front RGB-D camera for semantic navigation experiments -->
   <xacro:rgbd_camera_sensor gazebo="$(arg gazebo)" namespace="$(arg namespace)">
-    <origin xyz="0.135 0 ${0.135 + base_link_z_offset}" rpy="0 ${10*deg2rad} 0"/>
+    <origin xyz="0.155 0 ${0.055 + base_link_z_offset}" rpy="0 ${8*deg2rad} 0"/>
   </xacro:rgbd_camera_sensor>
   <xacro:if value="${'$(arg gazebo)' == 'classic'}">

File: create3_sim/irobot_create_common/irobot_create_description/urdf/sensors/rgbd_camera.urdf.xacro (robot description, xacro)
@@ -10,5 +10,5 @@
     <visual>
       <geometry>
-        <box size="0.055 0.09 0.035"/>
+        <box size="0.04 0.07 0.025"/>
       </geometry>
       <xacro:insert_block name="material_black"/>
@@ -16,8 +16,8 @@
     <collision>
       <geometry>
-        <box size="0.055 0.09 0.035"/>
+        <box size="0.04 0.07 0.025"/>
       </geometry>
     </collision>
-    <xacro:inertial_cuboid mass="0.08" x="0.055" y="0.09" z="0.035"/>
+    <xacro:inertial_cuboid mass="0.05" x="0.04" y="0.07" z="0.025"/>
   </link>
   <joint name="${name}_optical_joint" type="fixed">
@@ -34,5 +34,5 @@
       <always_on>true</always_on>
       <update_rate>${update_rate}</update_rate>
-      <visualize>true</visualize>
+      <visualize>false</visualize>
       <camera>
         <horizontal_fov>1.047</horizontal_fov>
